File: docs/Kicad/1000W Controller.kicad_sch (KiCad schematic)
At the start: 57 parts, among them Q2 Q_PMOS_GSD, Q3 Q_NMOS_GSD, U1 ADuM1201AR, U2 R-783.3-0.5, U3 LD1117V, U4 ADuM1201AR, U5 ADuM1201AR, U6 ADuM1201AR

Commit message: new
Parts:
- added R9: 10K, Resistor_SMD:R_0805_2012Metric, symbol Device:R
- renumbered Feather_M4_Express1 to Feather_M4_CAN_Express1
Connections:
- net ISO_GND: now also R9.1
- net remote_on_off: now also R9.2
Changed lines of the file:
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@@
 	(paper "A4")
 	(junction
+		(at 251.46 127)
+		(diameter 0)
+		(color 0 0 0 0)
+	)
+	(junction
 		(at 88.9 109.22)
 		(diameter 0)
@@
 	(wire
 		(pts
-			(xy 251.46 129.54) (xy 251.46 128.27)
+			(xy 251.46 129.54) (xy 251.46 127)
 		)
 		(stroke
@@
 	(wire
 		(pts
-			(xy 266.7 133.35) (xy 266.7 128.27)
+			(xy 266.7 133.35) (xy 266.7 127)
 		)
 		(stroke
@@
 	(wire
 		(pts
-			(xy 251.46 128.27) (xy 266.7 128.27)
+			(xy 251.46 127) (xy 266.7 127)
 		)
 		(stroke
@@
 	)
 	(label "remote_on_off"
-		(at 265.43 128.27 180)
+		(at 265.43 127 180)
 		(effects
 			(font
@@
 	(symbol
 		(lib_id "Breakout boards:ISO_GND")
+		(at 243.84 127 270)
+		(unit 1)
+		(exclude_from_sim no)
+		(in_bom yes)
+		(on_board yes)
+		(dnp no)
+		(property "Reference" "#PWR067"
+			(at 237.49 127 0)
+			(effects
+				(font
+					(size 1.27 1.27)
+				)
+				(hide yes)
+			)
+		)
+		(property "Value" "ISO_GND"
+			(at 232.664 126.492 90)
+			(effects
+				(font
+					(size 1.27 1.27)
+				)
+				(justify left)
+			)
+		)
+		(property "Footprint" ""
+			(at 243.84 127 0)
+			(effects
+				(font
+					(size 1.27 1.27)
+				)
+				(hide yes)
+			)
+		)
+		(property "Datasheet" ""
+			(at 243.84 127 0)
+			(effects
+				(font
+					(size 1.27 1.27)
+				)
+				(hide yes)
+			)
+		)
+		(property "Description" "Power symbol creates a global label with name \"GND\" , ground"
+			(at 243.84 127 0)
+			(effects
+				(font
+					(size 1.27 1.27)
+				)
+				(hide yes)
+			)
+		)
+		(pin "1"
+		)
+		(instances
+			(project "1000W Controller"
+				(path "/fb8df8b8-faed-4b3a-9fdd-17da7575274d"
+					(reference "#PWR067")
+					(unit 1)
+				)
+			)
+		)
+	)
+	(symbol
+		(lib_id "Breakout boards:ISO_GND")
 		(at 214.63 62.23 0)
 		(unit 1)
@@
 		(on_board yes)
 		(dnp no)
-		(property "Reference" "Feather_M4_Express1"
+		(property "Reference" "Feather_M4_CAN_Express1"
 			(at 173.5933 149.86 0)
 			(effects
@@
 			(project ""
 				(path "/fb8df8b8-faed-4b3a-9fdd-17da7575274d"
-					(reference "Feather_M4_Express1")
+					(reference "Feather_M4_CAN_Express1")
 					(unit 1)
 				)
@@
 					(unit 1)
 				)
+			)
+		)
+	)
+	(symbol
+		(lib_id "Device:R")
+		(at 247.65 127 90)
+		(unit 1)
+		(exclude_from_sim no)
+		(in_bom yes)
+		(on_board yes)
+		(dnp no)
+		(property "Reference" "R9"
+			(at 247.396 124.714 90)
+			(effects
+				(font
+					(size 1.27 1.27)
+				)
+			)
+		)
+		(property "Value" "10K"
+			(at 247.65 129.286 90)
+			(effects
+				(font
+					(size 1.27 1.27)
+				)
+			)
+		)
+		(property "Footprint" "Resistor_SMD:R_0805_2012Metric"
+			(at 247.65 128.778 90)
+			(effects
+				(font
+					(size 1.27 1.27)
+				)
+				(hide yes)
+			)
+		)
+		(property "Datasheet" "~"
+			(at 247.65 127 0)
+			(effects
+				(font
+					(size 1.27 1.27)
+				)
+				(hide yes)
+			)
+		)
+		(property "Description" "Resistor"
+			(at 247.65 127 0)
+			(effects
+				(font
+					(size 1.27 1.27)
+				)
+				(hide yes)
+			)
+		)
+		(pin "1"
+		)
+		(pin "2"
+		)
+		(instances
+			(project "1000W Controller"
+				(path "/fb8df8b8-faed-4b3a-9fdd-17da7575274d"
+					(reference "R9")
+					(unit 1)
+				)
